Commit message: Update sfixedlim.urdf

File: gym_Surena_v1/envs/SURENA/sfixedlim.urdf (robot description, URDF)
Before this commit: robot rrbot, 29 links, 28 joints
Joints:
- joint LLeg_AnkleP_J5: limit lower=-1.0 upper=1.3 effort=400 velocity=10.5 -> lower=-1.0 upper=1.3 effort=600 velocity=10.5
- joint LLeg_AnkleR_J6: limit lower=-0.7 upper=0.4 effort=400 velocity=10.5 -> lower=-0.7 upper=0.4 effort=600 velocity=10.5
- joint LLeg_HipP_J3: limit lower=-1.0 upper=1.2 effort=400 velocity=10.5 -> lower=-1.0 upper=1.2 effort=600 velocity=10.5
- joint LLeg_HipR_J2: limit lower=-0.1 upper=0.5 effort=400 velocity=10.5 -> lower=-0.1 upper=0.5 effort=600 velocity=10.5
- joint LLeg_HipY_J1: limit lower=-0.4 upper=1.0 effort=400 velocity=10.5 -> lower=-0.4 upper=1.0 effort=600 velocity=10.5
- joint LLeg_KneeP_J4: limit lower=0.0 upper=2.0 effort=400 velocity=10.5 -> lower=0.0 upper=2.0 effort=600 velocity=10.5
- joint RLeg_AnkleP_J5: limit lower=-1.0 upper=1.3 effort=400 velocity=10.5 -> lower=-1.0 upper=1.3 effort=600 velocity=10.5
- joint RLeg_AnkleR_J6: limit lower=-0.7 upper=0.7 effort=400 velocity=10.5 -> lower=-0.7 upper=0.7 effort=600 velocity=10.5
- joint RLeg_HipP_J3: limit lower=-1.0 upper=1.2 effort=400 velocity=10.5 -> lower=-1.0 upper=1.2 effort=600 velocity=10.5
- joint RLeg_HipR_J2: limit lower=-0.5 upper=0.1 effort=400 velocity=10.5 -> lower=-0.5 upper=0.1 effort=600 velocity=10.5
- joint RLeg_HipY_J1: limit lower=-1.0 upper=0.4 effort=400 velocity=10.5 -> lower=-1.0 upper=0.4 effort=600 velocity=10.5
- joint RLeg_KneeP_J4: limit lower=0.0 upper=2.0 effort=400 velocity=10.5 -> lower=0.0 upper=2.0 effort=600 velocity=10.5
